File: cmos-oscillator.sch (KiCad schematic (older format))
At the start: 24 parts

Commit message: added 74LS163 and connected vcc and ground
Parts:
- added U?: 74LS163, symbol 74LS163
Connections:
- wire segments 32 -> 33
Changed lines of the file:
@@
 LIBS:contrib
 LIBS:valves
-LIBS:cmos-oscillator-cache
 EELAYER 25 0
 EELAYER END
@@
 Text Label 3900 4300 0    60   ~ 0
 tempo
+$Comp
+L 74LS163 U?
+U 1 1 550FABA1
+P 7250 2400
+F 0 "U?" H 7300 2500 60  0000 C CNN
+F 1 "74LS163" H 7350 2200 60  0000 C CNN
+F 2 "" H 7250 2400 60  0000 C CNN
+F 3 "" H 7250 2400 60  0000 C CNN
+	1    7250 2400
+	1    0    0    -1
+$EndComp
+$Comp
+L VCC #PWR?
+U 1 1 550FAD69
+P 6950 1850
+F 0 "#PWR?" H 6950 1700 50  0001 C CNN
+F 1 "VCC" H 6950 2000 50  0000 C CNN
+F 2 "" H 6950 1850 60  0000 C CNN
+F 3 "" H 6950 1850 60  0000 C CNN
+	1    6950 1850
+	1    0    0    -1
+$EndComp
+$Comp
+L GND #PWR?
+U 1 1 550FAEF7
+P 6950 3000
+F 0 "#PWR?" H 6950 3000 30  0001 C CNN
+F 1 "GND" H 6950 2930 30  0001 C CNN
+F 2 "" H 6950 3000 60  0000 C CNN
+F 3 "" H 6950 3000 60  0000 C CNN
+	1    6950 3000
+	1    0    0    -1
+$EndComp
+Wire Wire Line
+	6950 2950 6950 3000
 $EndSCHEMATC
