File: cmos-oscillator.sch (KiCad schematic (older format))
At the start: 23 parts

Commit message: more work
Parts:
- removed C? (x5): C, symbol C
- removed R? (x5): RVAR 20k, symbol RVAR
- added C? (x5): C, symbol C
- added R? (x6): RVAR 20k, symbol RVAR
Connections:
- net GND: now also C?.1, C?.1, C?.1, C?.1, C?.1
- net in1: now reaches U?.1
- net in1: now also U?.12, C?.2, R?.1, R?.2
- net amp: now reaches U?.2
- net amp: now also U?.4, U?.6, R?.2, R?.2, R?.2
- net in2: now reaches U?.3
- net in2: now also U?.10, C?.2, R?.1, R?.2
- net in3: now reaches U?.5
- net in3: now also C?.2, R?.1
- net in4: now reaches U?.9
- net in4: now also C?.2, R?.1
- net clock: now reaches U?.8
- net clock: now also R?.2
- net in5: now reaches U?.11
- net in5: now also C?.2, R?.1
- net in6: now reaches C?.2, U?.13
- net in6: now also R?.1; no longer R?.2
- net at R?.1: no longer U?.12

Commit message: changed some values
Parts:
- 20k: renamed from R?; value RVAR 20k -> RVAR
- gave numbers to parts that had none: 1
Changed lines of the file:
@@
 $EndComp
 $Comp
-L VCC #PWR?
+L VCC #PWR01
 U 1 1 550CCCEB
 P 3450 1750
-F 0 "#PWR?" H 3450 1600 50  0001 C CNN
+F 0 "#PWR01" H 3450 1600 50  0001 C CNN
 F 1 "VCC" H 3450 1900 50  0000 C CNN
 F 2 "" H 3450 1750 60  0000 C CNN
@@
 $EndComp
 $Comp
-L GND #PWR?
+L GND #PWR02
 U 1 1 550CCEA3
 P 3450 5200
-F 0 "#PWR?" H 3450 4950 50  0001 C CNN
+F 0 "#PWR02" H 3450 4950 50  0001 C CNN
 F 1 "GND" H 3450 5050 50  0000 C CNN
 F 2 "" H 3450 5200 60  0000 C CNN
@@
 	3450 3500 3450 5200
 $Comp
-L C C?
+L C 2.7nf
 U 1 1 550CB6A2
 P 4450 1850
-F 0 "C?" H 4475 1950 50  0000 L CNN
+F 0 "2.7nf" H 4475 1950 50  0000 L CNN
 F 1 "C" H 4475 1750 50  0000 L CNN
 F 2 "" H 4488 1700 30  0000 C CNN
@@
 $EndComp
 $Comp
-L GND #PWR?
+L GND #PWR03
 U 1 1 550CB6A8
 P 4600 1850
-F 0 "#PWR?" H 4600 1600 50  0001 C CNN
+F 0 "#PWR03" H 4600 1600 50  0001 C CNN
 F 1 "GND" H 4600 1700 50  0000 C CNN
 F 2 "" H 4600 1850 60  0000 C CNN
@@
 $EndComp
 $Comp
-L RVAR R?
+L RVAR 20k
 U 1 1 550E512D
 P 4300 2400
-F 0 "R?" V 4380 2350 50  0000 C CNN
-F 1 "RVAR 20k" V 4220 2460 50  0000 C CNN
+F 0 "20k" V 4380 2350 50  0000 C CNN
+F 1 "RVAR" V 4220 2460 50  0000 C CNN
 F 2 "" H 4300 2400 60  0000 C CNN
 F 3 "" H 4300 2400 60  0000 C CNN
@@
 in1
 $Comp
-L C C?
+L C 2.7nf
 U 1 1 550E5610
 P 4450 3000
-F 0 "C?" H 4475 3100 50  0000 L CNN
+F 0 "2.7nf" H 4475 3100 50  0000 L CNN
 F 1 "C" H 4475 2900 50  0000 L CNN
 F 2 "" H 4488 2850 30  0000 C CNN
@@
 $EndComp
 $Comp
-L GND #PWR?
+L GND #PWR04
 U 1 1 550E5616
 P 4600 3000
-F 0 "#PWR?" H 4600 2750 50  0001 C CNN
+F 0 "#PWR04" H 4600 2750 50  0001 C CNN
 F 1 "GND" H 4600 2850 50  0000 C CNN
 F 2 "" H 4600 3000 60  0000 C CNN
@@
 	4300 3000 3800 3000
 $Comp
-L RVAR R?
+L RVAR 20k
 U 1 1 550E561D
 P 4300 3550
-F 0 "R?" V 4380 3500 50  0000 C CNN
-F 1 "RVAR 20k" V 4220 3610 50  0000 C CNN
+F 0 "20k" V 4380 3500 50  0000 C CNN
+F 1 "RVAR" V 4220 3610 50  0000 C CNN
 F 2 "" H 4300 3550 60  0000 C CNN
 F 3 "" H 4300 3550 60  0000 C CNN
@@
 in2
 $Comp
-L C C?
+L C 2.7nf
 U 1 1 550E57D0
 P 4450 4150
-F 0 "C?" H 4475 4250 50  0000 L CNN
+F 0 "2.7nf" H 4475 4250 50  0000 L CNN
 F 1 "C" H 4475 4050 50  0000 L CNN
 F 2 "" H 4488 4000 30  0000 C CNN
@@
 $EndComp
 $Comp
-L GND #PWR?
+L GND #PWR05
 U 1 1 550E57D6
 P 4600 4150
-F 0 "#PWR?" H 4600 3900 50  0001 C CNN
+F 0 "#PWR05" H 4600 3900 50  0001 C CNN
 F 1 "GND" H 4600 4000 50  0000 C CNN
 F 2 "" H 4600 4150 60  0000 C CNN
@@
 	4300 4150 3800 4150
 $Comp
-L RVAR R?
+L RVAR 20k
 U 1 1 550E57DD
 P 4300 4700
-F 0 "R?" V 4380 4650 50  0000 C CNN
-F 1 "RVAR 20k" V 4220 4760 50  0000 C CNN
+F 0 "20k" V 4380 4650 50  0000 C CNN
+F 1 "RVAR" V 4220 4760 50  0000 C CNN
 F 2 "" H 4300 4700 60  0000 C CNN
 F 3 "" H 4300 4700 60  0000 C CNN
@@
 clock
 $Comp
-L C C?
+L C 2.7nf
 U 1 1 550E5AF4
 P 2450 3000
-F 0 "C?" H 2475 3100 50  0000 L CNN
+F 0 "2.7nf" H 2475 3100 50  0000 L CNN
 F 1 "C" H 2475 2900 50  0000 L CNN
 F 2 "" H 2488 2850 30  0000 C CNN
@@
 $EndComp
 $Comp
-L GND #PWR?
+L GND #PWR06
 U 1 1 550E5AFA
 P 2300 3000
-F 0 "#PWR?" H 2300 2750 50  0001 C CNN
+F 0 "#PWR06" H 2300 2750 50  0001 C CNN
 F 1 "GND" H 2300 2850 50  0000 C CNN
 F 2 "" H 2300 3000 60  0000 C CNN
@@
 	2600 3000 3100 3000
 $Comp
-L RVAR R?
+L RVAR 20k
 U 1 1 550E5B01
 P 2600 3550
-F 0 "R?" V 2680 3500 50  0000 C CNN
-F 1 "RVAR 20k" V 2520 3610 50  0000 C CNN
+F 0 "20k" V 2680 3500 50  0000 C CNN
+F 1 "RVAR" V 2520 3610 50  0000 C CNN
 F 2 "" H 2600 3550 60  0000 C CNN
 F 3 "" H 2600 3550 60  0000 C CNN
@@
 amp
 $Comp
-L C C?
+L C 2.7nf
 U 1 1 550E5B0C
 P 2450 4150
-F 0 "C?" H 2475 4250 50  0000 L CNN
+F 0 "2.7nf" H 2475 4250 50  0000 L CNN
 F 1 "C" H 2475 4050 50  0000 L CNN
 F 2 "" H 2488 4000 30  0000 C CNN
@@
 $EndComp
 $Comp
-L GND #PWR?
+L GND #PWR07
 U 1 1 550E5B12
 P 2300 4150
-F 0 "#PWR?" H 2300 3900 50  0001 C CNN
+F 0 "#PWR07" H 2300 3900 50  0001 C CNN
 F 1 "GND" H 2300 4000 50  0000 C CNN
 F 2 "" H 2300 4150 60  0000 C CNN
@@
 	2600 4150 3100 4150
 $Comp
-L RVAR R?
+L RVAR 20k
 U 1 1 550E5B19
 P 2600 4700
-F 0 "R?" V 2680 4650 50  0000 C CNN
-F 1 "RVAR 20k" V 2520 4760 50  0000 C CNN
+F 0 "20k" V 2680 4650 50  0000 C CNN
+F 1 "RVAR" V 2520 4760 50  0000 C CNN
 F 2 "" H 2600 4700 60  0000 C CNN
 F 3 "" H 2600 4700 60  0000 C CNN
@@
 Connection ~ 4300 1850
 $Comp
-L C C?
+L C 2.7nf
 U 1 1 550E51D2
 P 2450 1850
-F 0 "C?" H 2475 1950 50  0000 L CNN
+F 0 "2.7nf" H 2475 1950 50  0000 L CNN
 F 1 "C" H 2475 1750 50  0000 L CNN
 F 2 "" H 2488 1700 30  0000 C CNN
@@
 $EndComp
 $Comp
-L GND #PWR?
+L GND #PWR08
 U 1 1 550E51D8
 P 2300 1850
-F 0 "#PWR?" H 2300 1600 50  0001 C CNN
+F 0 "#PWR08" H 2300 1600 50  0001 C CNN
 F 1 "GND" H 2300 1700 50  0000 C CNN
 F 2 "" H 2300 1850 60  0000 C CNN
@@
 $EndComp
 $Comp
-L RVAR R?
+L RVAR 20k
 U 1 1 550E51DF
 P 2600 2400
-F 0 "R?" V 2680 2350 50  0000 C CNN
-F 1 "RVAR 20k" V 2520 2460 50  0000 C CNN
+F 0 "20k" V 2680 2350 50  0000 C CNN
+F 1 "RVAR" V 2520 2460 50  0000 C CNN
 F 2 "" H 2600 2400 60  0000 C CNN
 F 3 "" H 2600 2400 60  0000 C CNN
